File: colorTemp.brd (EAGLE design)
At the start: 100 x 80 mm, 21 parts, among them IC1 STM32F10XCXT6

Commit message: Board update
Parts:
- moved R2 51.7 mm to (44.5, 36.7), turned to 90 degrees
- moved JP5 47.7 mm to (44.5, 58.5)
- moved R4 35.2 mm to (58.8, 42.5), turned to 270 degrees
- moved JP1 4.12 mm to (56.3, 58.7)
- moved JP2 2.67 mm to (62.4, 19.1)
- moved JP3 2.44 mm to (41.3, 48.5)
- moved JP4 1.91 mm to (41.3, 35.6)
- moved C2 0.76 mm to (49.5, 46.4)
Routing:
- net 3V3: track 0.00 -> 100.2 mm, vias 0 -> 4
- net OUT: track 0.00 -> 89.4 mm
- net N$20: track 0.00 -> 24.6 mm
- net SWCLK: track 0.00 -> 23.8 mm
- net RESET: track 0.00 -> 19.8 mm
- net SWDIO: track 0.00 -> 18.5 mm
- net RX: track 0.00 -> 18.3 mm
- net GND: track 0.00 -> 18.1 mm
- net TX: track 0.00 -> 13.8 mm
- net OE: track 0.00 -> 11.7 mm
- net S3: track 0.00 -> 10.3 mm
- net S2: track 0.76 -> 9.22 mm
- net S1: track 0.00 -> 7.24 mm
- net S0: track 0.00 -> 6.40 mm
- net N$2: track 0.00 -> 4.16 mm
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- added copper zone on layer 1, net 3V3
- added copper zone on layer 1, net GND
